File: hall-current-probe.kicad_pcb (KiCad board)
At the start: 2 copper layers, 64 x 30 mm, 31 parts, among them J1 USB, J2 CONN-SMA-5-1814400-1, J3 CONN-SMA-5-1814400-1, J4 2834076-1, J5 2834076-1, U1 ACS730, U2 ACS730, U3 MC33078D, U4 LMC7660

Commit message: Fix ERC and BOM issues
Parts:
- C1, C4: value 150pF -> 100pF
- J2, J3: value CONN-SMA-5-1814400-1 -> CONN-SMA
Changed lines of the file:
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@@
-(kicad_pcb (version 20171130) (host pcbnew "(5.0.0-rc2-21-g8f5cb3259)")
+(kicad_pcb (version 20171130) (host pcbnew "(5.0.0-rc2-204-g01c2d93a8)")
   (general
     (thickness 1.6)
@@
       (hpglpennumber 1)
       (hpglpenspeed 20)
-      (hpglpendiameter 15)
+      (hpglpendiameter 15.000000)
       (psnegative false)
       (psa4output false)
@@
       (outputformat 1)
       (mirror false)
-      (drillshape 1)
+      (drillshape 0)
       (scaleselection 1)
-      (outputdirectory ""))
+      (outputdirectory "fabrication/gerbers"))
   )
   (net 0 "")
@@
     (at 22.5 4.25 180)
     (attr smd)
-    (fp_text reference J2 (at 0 -4.75 180) (layer F.SilkS)
-      (effects (font (size 0.8 0.8) (thickness 0.15)))
-    )
-    (fp_text value CONN-SMA-5-1814400-1 (at 0 0 180) (layer F.Fab)
+    (fp_text reference J2 (at -4.75 2.5 270) (layer F.SilkS)
+      (effects (font (size 0.8 0.8) (thickness 0.15)))
+    )
+    (fp_text value CONN-SMA (at 0 0 180) (layer F.Fab)
       (effects (font (size 0.8 0.8) (thickness 0.15)))
     )
@@
     (at 41.5 4.25 180)
     (attr smd)
-    (fp_text reference J3 (at 0 -4.75 180) (layer F.SilkS)
-      (effects (font (size 0.8 0.8) (thickness 0.15)))
-    )
-    (fp_text value CONN-SMA-5-1814400-1 (at 0 0 180) (layer F.Fab)
+    (fp_text reference J3 (at -4.75 2.5 270) (layer F.SilkS)
+      (effects (font (size 0.8 0.8) (thickness 0.15)))
+    )
+    (fp_text value CONN-SMA (at 0 0 180) (layer F.Fab)
       (effects (font (size 0.8 0.8) (thickness 0.15)))
     )
@@
       (effects (font (size 0.8 0.8) (thickness 0.15)))
     )
-    (fp_text value 150pF (at 0 0 270) (layer F.Fab)
+    (fp_text value 100pF (at 0 0 270) (layer F.Fab)
       (effects (font (size 0.5 0.5) (thickness 0.1)))
     )
@@
       (effects (font (size 0.8 0.8) (thickness 0.15)))
     )
-    (fp_text value 150pF (at 0 0 270) (layer F.Fab)
+    (fp_text value 100pF (at 0 0 270) (layer F.Fab)
       (effects (font (size 0.5 0.5) (thickness 0.1)))
     )
@@
   (segment (start 47.2 25) (end 46.15 25) (width 0.6) (layer F.Cu) (net 19))
   (segment (start 47.865 24.335) (end 47.2 25) (width 0.6) (layer F.Cu) (net 19))
+  (via (at 47.5 22.75) (size 0.8) (drill 0.4) (layers F.Cu B.Cu) (net 19))
+  (via (at 47.5 25.75) (size 0.8) (drill 0.4) (layers F.Cu B.Cu) (net 19))
+  (via (at 46.25 27) (size 0.8) (drill 0.4) (layers F.Cu B.Cu) (net 19))
+  (via (at 46.25 25.75) (size 0.8) (drill 0.4) (layers F.Cu B.Cu) (net 19))
+  (via (at 47.5 27.25) (size 0.8) (drill 0.4) (layers F.Cu B.Cu) (net 19))
+  (via (at 47.5 24.25) (size 0.8) (drill 0.4) (layers F.Cu B.Cu) (net 19))
+  (segment (start 46 27.25) (end 46.25 27) (width 0.25) (layer F.Cu) (net 19))
+  (segment (start 46 28.5) (end 46 27.25) (width 2.2) (layer F.Cu) (net 19))
   (segment (start 18.25 25) (end 23 25) (width 0.6) (layer F.Cu) (net 20))
   (segment (start 16.75 25) (end 18.25 25) (width 0.6) (layer F.Cu) (net 20))
@@
   (segment (start 17.405 22.405) (end 17.75 22.75) (width 0.6) (layer F.Cu) (net 20))
   (segment (start 17.405 21.2) (end 17.405 22.405) (width 0.6) (layer F.Cu) (net 20))
-  (via (at 50.75 27) (size 0.8) (drill 0.4) (layers F.Cu B.Cu) (net 22))
-  (via (at 49.5 22.75) (size 0.8) (drill 0.4) (layers F.Cu B.Cu) (net 22))
-  (via (at 49.5 27.25) (size 0.8) (drill 0.4) (layers F.Cu B.Cu) (net 22))
-  (via (at 49.5 25.75) (size 0.8) (drill 0.4) (layers F.Cu B.Cu) (net 22))
-  (via (at 49.5 24.25) (size 0.8) (drill 0.4) (layers F.Cu B.Cu) (net 22))
-  (via (at 50.75 25.75) (size 0.8) (drill 0.4) (layers F.Cu B.Cu) (net 22))
+  (segment (start 18 28.5) (end 18 27.25) (width 2.2) (layer F.Cu) (net 20))
   (segment (start 13.595 24.155) (end 13.25 24.25) (width 0.6) (layer F.Cu) (net 21))
   (segment (start 12.75 25) (end 4 25) (width 0.6) (layer F.Cu) (net 21))
@@
   (segment (start 13.595 22.405) (end 13.25 22.75) (width 0.6) (layer F.Cu) (net 21))
   (segment (start 13.595 21.2) (end 13.595 22.405) (width 0.6) (layer F.Cu) (net 21))
-  (via (at 47.5 22.75) (size 0.8) (drill 0.4) (layers F.Cu B.Cu) (net 19))
-  (via (at 47.5 25.75) (size 0.8) (drill 0.4) (layers F.Cu B.Cu) (net 19))
-  (via (at 46.25 27) (size 0.8) (drill 0.4) (layers F.Cu B.Cu) (net 19))
-  (via (at 46.25 25.75) (size 0.8) (drill 0.4) (layers F.Cu B.Cu) (net 19))
-  (via (at 47.5 27.25) (size 0.8) (drill 0.4) (layers F.Cu B.Cu) (net 19))
-  (via (at 47.5 24.25) (size 0.8) (drill 0.4) (layers F.Cu B.Cu) (net 19))
-  (segment (start 46 27.25) (end 46.25 27) (width 0.25) (layer F.Cu) (net 19))
-  (segment (start 46 28.5) (end 46 27.25) (width 2.2) (layer F.Cu) (net 19))
+  (segment (start 13 28.5) (end 13 27.25) (width 2.2) (layer F.Cu) (net 21))
+  (via (at 50.75 27) (size 0.8) (drill 0.4) (layers F.Cu B.Cu) (net 22))
+  (via (at 49.5 22.75) (size 0.8) (drill 0.4) (layers F.Cu B.Cu) (net 22))
+  (via (at 49.5 27.25) (size 0.8) (drill 0.4) (layers F.Cu B.Cu) (net 22))
+  (via (at 49.5 25.75) (size 0.8) (drill 0.4) (layers F.Cu B.Cu) (net 22))
+  (via (at 49.5 24.25) (size 0.8) (drill 0.4) (layers F.Cu B.Cu) (net 22))
+  (via (at 50.75 25.75) (size 0.8) (drill 0.4) (layers F.Cu B.Cu) (net 22))
   (segment (start 49.135 21.2) (end 49.135 24.285) (width 0.6) (layer F.Cu) (net 22))
   (segment (start 49.85 25) (end 58 25) (width 0.6) (layer F.Cu) (net 22))
@@
   (segment (start 51 27.25) (end 50.75 27) (width 0.25) (layer F.Cu) (net 22))
   (segment (start 51 28.5) (end 51 27.25) (width 2.2) (layer F.Cu) (net 22))
-  (segment (start 18 28.5) (end 18 27.25) (width 2.2) (layer F.Cu) (net 20))
-  (segment (start 13 28.5) (end 13 27.25) (width 2.2) (layer F.Cu) (net 21))
   (zone (net 2) (net_name GND) (layer B.Cu) (hatch edge 0.508)
     (connect_pads (clearance 0.3))
