File: hall-current-probe.sch (KiCad schematic (older format))
At the start: 31 parts, among them J1 USB, J2 CONN-SMA-5-1814400-1, J3 CONN-SMA-5-1814400-1, J4 2834076-1, J5 2834076-1, U1 ACS730, U2 ACS730, U3 MC33078D, U4 LMC7660

Commit message: Update library
Parts:
- J2, J3: value CONN-SMA-5-1814400-1 -> CONN-SMA
- U1, U2: symbol AMS:ACS730 -> Allegro:ACS730; BOM AMS ACS730CTR-20AB-T -> Allegro ACS730KLCTR-xxAB-T; MPN (none) -> ACS730KLCTR-xxAB-T; Manuf (none) -> Allegro
Changed lines of the file:
@@
 encoding utf-8
 Sheet 1 1
-Title ""
-Date ""
-Rev ""
-Comp ""
+Title "Dual Channel Hall Current Oscilloscope Probe"
+Date "2018-06-24"
+Rev "1.0"
+Comp "Electrum EE"
 Comment1 ""
 Comment2 ""
@@
 $EndComp
 $Comp
-L AMS:ACS730 U1
+L Allegro:ACS730 U1
 U 1 1 5B2EC1E2
 P 4600 2250
-F 0 "U1" H 4600 2939 60  0000 C CNN
-F 1 "ACS730" H 4600 2833 60  0000 C CNN
-F 2 "IPC7351-Nominal:SOIC127P600X175-8" H 4400 2250 60  0001 C CNN
-F 3 "" H 4400 2250 60  0001 C CNN
-F 4 "AMS ACS730CTR-20AB-T" H -550 0   50  0001 C CNN "BOM"
+F 0 "U1" H 4600 2917 50  0000 C CNN
+F 1 "ACS730" H 4600 2826 50  0000 C CNN
+F 2 "IPC7351-Nominal:SOIC127P600X175-8" H 4600 1550 50  0001 C CNN
+F 3 "https://www.allegromicro.com/~/media/Files/Datasheets/ACS730-Datasheet.ashx" H 4600 1650 50  0001 C CNN
+F 4 "Allegro ACS730KLCTR-xxAB-T" H -550 0   50  0001 C CNN "BOM"
+F 5 "ACS730KLCTR-xxAB-T" H 0   0   50  0001 C CNN "MPN"
+F 6 "Allegro" H 0   0   50  0001 C CNN "Manuf"
 	1    4600 2250
 	1    0    0    -1
@@
 $EndComp
 $Comp
-L AMS:ACS730 U2
+L Allegro:ACS730 U2
 U 1 1 5B2EEA3E
 P 4600 4500
-F 0 "U2" H 4600 5189 60  0000 C CNN
-F 1 "ACS730" H 4600 5083 60  0000 C CNN
-F 2 "IPC7351-Nominal:SOIC127P600X175-8" H 4400 4500 60  0001 C CNN
-F 3 "" H 4400 4500 60  0001 C CNN
-F 4 "AMS ACS730CTR-20AB-T" H -550 0   50  0001 C CNN "BOM"
+F 0 "U2" H 4600 5167 50  0000 C CNN
+F 1 "ACS730" H 4600 5076 50  0000 C CNN
+F 2 "IPC7351-Nominal:SOIC127P600X175-8" H 4600 3800 50  0001 C CNN
+F 3 "https://www.allegromicro.com/~/media/Files/Datasheets/ACS730-Datasheet.ashx" H 4600 3900 50  0001 C CNN
+F 4 "Allegro ACS730KLCTR-xxAB-T" H -550 0   50  0001 C CNN "BOM"
+F 5 "ACS730KLCTR-xxAB-T" H 0   0   50  0001 C CNN "MPN"
+F 6 "Allegro" H 0   0   50  0001 C CNN "Manuf"
 	1    4600 4500
 	1    0    0    -1
@@
 P 8400 2350
 F 0 "J2" H 8300 2376 50  0000 R CNN
-F 1 "CONN-SMA-5-1814400-1" H 8300 2285 50  0000 R CNN
+F 1 "CONN-SMA" H 8300 2285 50  0000 R CNN
 F 2 "manuf:CONN-TE-1814400" H 8400 2350 50  0001 C CNN
 F 3 "" H 8400 2350 50  0000 C CNN
@@
 P 8400 4600
 F 0 "J3" H 8300 4626 50  0000 R CNN
-F 1 "CONN-SMA-5-1814400-1" H 8300 4535 50  0000 R CNN
+F 1 "CONN-SMA" H 8300 4535 50  0000 R CNN
 F 2 "manuf:CONN-TE-1814400" H 8400 4600 50  0001 C CNN
 F 3 "" H 8400 4600 50  0000 C CNN

Commit message: Fix ERC and BOM issues
Parts:
- C1, C4: value 150pF -> 100pF; BOM CAP MLCC 150pF C0G 50V 5% [0603] -> CAP MLCC 100pF C0G 50V [0603]; MPN (none) -> 500R14N101JV4T; Manuf (none) -> Johanson
- C10, C2, C5: BOM CAP MLCC 100nF C0G 50V 5% [0603] -> CAP MLCC 100nF X5R 50V [0603]; MPN (none) -> UMK107BJ104KAHT; Manuf (none) -> Taiyo Yuden
- C3, C6: BOM CAP MLCC 1nF C0G 50V 5% [0603] -> CAP MLCC 1nF C0G 25V [0603]; MPN (none) -> CC0603JRNPO8BN102; Manuf (none) -> Yageo
- C7, C8, C9: BOM CAP MLCC 10uF C0G 50V 5% [0805] -> CAP MLCC 10uF X5R 10V [0805]; MPN (none) -> LMK212BJ106KG-T; Manuf (none) -> Taiyo Yuden
- J1: BOM (none) -> CONN FCI 10118193-0001LF
- J2, J3: BOM (none) -> CONN SMA; MPN (none) -> DSMAF14155L; Manuf (none) -> Ebay
- J4, J5: BOM (none) -> CONN TE 2834076-1
- R1, R2, R3, R4, R5, R6, R7, R8: MPN (none) -> CR0603-FX-1002ELF; Manuf (none) -> Bourns
- U1, U2: BOM Allegro ACS730KLCTR-xxAB-T -> Allegro ACS730KLCTR-20AB-T; MPN ACS730KLCTR-xxAB-T -> ACS730KLCTR-20AB-T
- U3: BOM ONSEMI MC33078D -> TI MC33078DR; MPN (none) -> MC33078DR; Manuf (none) -> TI
Connections:
- wire segments 118 -> 122
- no-connect marks 2 -> 5
